File: RFM95_Serial_Converter_PCB/915MHz_Radio.kicad_sch (KiCad schematic)
At the start: 4 parts, among them U1 RFM95W-915S2

Commit message: Finalised component placement and board edge
Parts:
- AE1: LCSC (none) -> C496550
Changed lines of the file:
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@@
+      (effects (font (size 1.27 1.27)) hide)
+    )
+    (property "LCSC" "C496550" (id 4) (at 162.56 80.518 0)
       (effects (font (size 1.27 1.27)) hide)
     )
