File: RFM95_Serial_Converter_PCB/Data_Interfaces.kicad_sch (KiCad schematic)
At the start: 10 parts, among them J1 Conn_01x04, J2 SM06B-GHS-TB(LF)(SN), J3 SM06B-GHS-TB(LF)(SN), J4 USB_B_Micro, J5 USB_B_Micro, U3 USBLC6-2SC6, U4 USBLC6-2SC6, U5 CP2102N-Axx-xQFN28

Commit message: Routed and ready to order
Connections:
- net USB1_IN_D+: now reaches U3.6 (I/O1), U5.4 (D+)
- net USB1_IN_D-: now reaches U3.4 (I/O2), U5.5 (D-)
- net USB1_D-: now reaches J4.2 (D-), U3.3 (I/O2)
- net USB1_D+: now reaches J4.3 (D+), U3.1 (I/O1)
- net USB2_D-: now reaches J5.2 (D-), U4.3 (I/O2)
- net USB2_D+: now reaches J5.3 (D+), U4.1 (I/O1)
Changed lines of the file:
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@@
+    (effects (font (size 1.27 1.27)) (justify left bottom))
+  )
+  (label "USB1_IN_D+" (at 228.092 82.55 0)
+    (effects (font (size 1.27 1.27)) (justify left bottom))
+  )
+  (label "USB1_IN_D-" (at 228.092 80.01 0)
+    (effects (font (size 1.27 1.27)) (justify left bottom))
+  )
+  (label "USB2_D-" (at 192.024 133.858 0)
+    (effects (font (size 1.27 1.27)) (justify left bottom))
+  )
+  (label "USB1_D+" (at 192.024 71.628 0)
+    (effects (font (size 1.27 1.27)) (justify left bottom))
+  )
+  (label "USB1_D-" (at 192.024 91.948 0)
+    (effects (font (size 1.27 1.27)) (justify left bottom))
+  )
+  (label "USB2_D+" (at 192.024 113.538 0)
     (effects (font (size 1.27 1.27)) (justify left bottom))
   )
@@
     (in_bom yes) (on_board yes)
     (property "Reference" "U3" (id 0) (at 220.0797 77.1991 90))
-    (property "Value" "USBLC6-2SC6" (id 1) (at 204.089 70.358 90))
+    (property "Value" "USBLC6-2SC6" (id 1) (at 204.724 67.564 90))
     (property "Footprint" "Package_TO_SOT_SMD:SOT-23-6" (id 2) (at 192.024 81.788 0)
       (effects (font (size 1.27 1.27)) hide)

Commit message: Working code and PCBs
Other:
- note added: "TX and RX are suspected of being backwards"
Changed lines of the file:
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@@
+    (effects (font (size 1.27 1.27)) (justify left bottom))
+  )
+  (text "TX and RX are suspected\nof being backwards" (at 259.08 60.96 0)
     (effects (font (size 1.27 1.27)) (justify left bottom))
   )
